File: PicoPadV2.kicad_pcb (KiCad board)
At the start: 2 copper layers, 88.2 x 146 mm, 49 parts, among them SW1 CherryMX, SW10 CherryMX, SW11 CherryMX, SW12 CherryMX, SW13 CherryMX, SW14 CherryMX, SW15 CherryMX, SW16 CherryMX, SW17 CherryMX, SW18 CherryMX, SW19 CherryMX, SW2 CherryMX, SW20 CherryMX, SW3 CherryMX, SW4 RotaryEncoder_Switch, SW5 CherryMX, SW6 CherryMX, SW7 CherryMX, SW8 CherryMX, SW9 CherryMX, U1 Pico

Commit message: Add files via upload
Other:
- board text added: "https://github.com/jaredm577/PicoPad-V2"
